File: hardware/BugCON_2023.kicad_sch (KiCad schematic)
At the start: 30 parts, among them J1 Conn_01x04_Pin, J2 Conn_01x04_Pin, J3 Conn_01x02, P1 USB_C_Plug_USB2.0, Q1 DMG3415U-7, SW1 RESET, SW2 GPIO, SW3 ON, U1 ESP32-S3-WROOM-1U-N16, U2 AP2112K-3.3

Commit message: Add_PCB
Parts:
- D2, D6, D7, D8: footprint Ekoparty:LED_SK6812MINI_PLCC4_3.5x3.5mm_P1.75mm -> FootprintsB:WS2812B_WDS
- P1: footprint Connectors:C393939 -> Connector_USB:USB_C_Receptacle_G-Switch_GT-USB-7010ASV
- U1: footprint RF_Module:ESP32-S3-WROOM-1U -> FootprintsB:XCVR_ESP32-S3-WROOM-1-N8R2; manf# ESP32-S3-WROOM-1U-N16 -> ESP32-S3-WROOM-1-N4
Connections:
- net PIN: now also U1.31 (IO38); no longer U1.26 (IO45)
Changed lines of the file:
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@@
   (no_connect (at 156.337 40.132))
   (no_connect (at 196.977 32.512))
-  (no_connect (at 196.977 52.832))
+  (no_connect (at 200.787 65.532))
   (no_connect (at 156.337 47.752))
   (no_connect (at 196.977 47.752))
@@
     (stroke (width 0) (type default))
   )
+  (wire (pts (xy 199.136 52.832) (xy 196.977 52.832))
+    (stroke (width 0) (type default))
+  )
   (wire (pts (xy 84.582 125.222) (xy 84.582 127.381))
     (stroke (width 0) (type default))
@@
     (effects (font (size 1.27 1.27)) (justify left bottom))
   )
-  (label "PIN" (at 200.787 65.532 0) (fields_autoplaced)
+  (label "PIN" (at 199.136 52.832 0) (fields_autoplaced)
     (effects (font (size 1.27 1.27)) (justify left bottom))
   )
@@
       (effects (font (size 1.524 1.524)))
     )
-    (property "Footprint" "RF_Module:ESP32-S3-WROOM-1U" (at 176.657 21.336 0)
+    (property "Footprint" "FootprintsB:XCVR_ESP32-S3-WROOM-1-N8R2" (at 176.657 21.336 0)
       (effects (font (size 1.524 1.524)) hide)
     )
@@
       (effects (font (size 1.524 1.524)) hide)
     )
-    (property "manf#" "ESP32-S3-WROOM-1U-N16" (at 156.337 27.432 0)
+    (property "manf#" "ESP32-S3-WROOM-1-N4" (at 156.337 27.432 0)
       (effects (font (size 1.27 1.27)) hide)
     )
@@
       (effects (font (size 1.27 1.27)))
     )
-    (property "Footprint" "Ekoparty:LED_SK6812MINI_PLCC4_3.5x3.5mm_P1.75mm" (at 236.22 143.129 0)
+    (property "Footprint" "FootprintsB:WS2812B_WDS" (at 236.22 143.129 0)
       (effects (font (size 1.27 1.27)) (justify left top) hide)
     )
@@
       (effects (font (size 1.27 1.27)))
     )
-    (property "Footprint" "Ekoparty:LED_SK6812MINI_PLCC4_3.5x3.5mm_P1.75mm" (at 186.563 143.129 0)
+    (property "Footprint" "FootprintsB:WS2812B_WDS" (at 186.563 143.129 0)
       (effects (font (size 1.27 1.27)) (justify left top) hide)
     )
@@
       (effects (font (size 1.27 1.27)))
     )
-    (property "Footprint" "Ekoparty:LED_SK6812MINI_PLCC4_3.5x3.5mm_P1.75mm" (at 211.836 143.129 0)
+    (property "Footprint" "FootprintsB:WS2812B_WDS" (at 211.836 143.129 0)
       (effects (font (size 1.27 1.27)) (justify left top) hide)
     )
@@
       (effects (font (size 1.27 1.27)))
     )
-    (property "Footprint" "Connectors:C393939" (at 30.734 36.576 0)
+    (property "Footprint" "Connector_USB:USB_C_Receptacle_G-Switch_GT-USB-7010ASV" (at 30.734 36.576 0)
       (effects (font (size 1.27 1.27)) hide)
     )
@@
       (effects (font (size 1.27 1.27)))
     )
-    (property "Footprint" "Ekoparty:LED_SK6812MINI_PLCC4_3.5x3.5mm_P1.75mm" (at 260.223 143.129 0)
+    (property "Footprint" "FootprintsB:WS2812B_WDS" (at 260.223 143.129 0)
       (effects (font (size 1.27 1.27)) (justify left top) hide)
     )
