File: hardware/SAMD11/BugCON2023_samd11.kicad_sch (KiCad schematic)
At the start: 30 parts, among them J1 Conn_01x04_Pin, J2 Conn_01x04_Pin, J3 PAD2, J4 PAD, P1 USB_C_Plug_USB2.0, Q1 DMG3415U-7, SW1 SW_Push, SW2 ON, U1 ATSAMD11C14A-SS, U2 AP2112K-3.3

Commit message: add serial on SAMD11
Parts:
- removed J2: Conn_01x04_Pin, Connector_PinSocket_2.54mm:PinSocket_1x04_P2.54mm_Vertical, symbol Connector:Conn_01x04_Pin
- added J5: Serial, Connector_PinSocket_2.54mm:PinSocket_1x03_P2.54mm_Vertical, symbol Connector:Conn_01x03_Pin
- J1: value Conn_01x04_Pin -> I2C; now not fitted
Connections:
- net GND: now also J5.3 (Pin_3)
- net RX: now also U1.3 (PA09/XOUT), J5.1 (Pin_1)
- net TX: now also U1.2 (PA08/XIN), J5.2 (Pin_2)
- no-connect marks 3 -> 1
Other:
- moved on the sheet: U1
