File: hardware/SAMD11/BugCON2023_samd11.kicad_pcb (KiCad board)
At the start: 2 copper layers, 122.4 x 97.9 mm, 67 parts, among them J1 I2C, J5 Serial, P1 USB_C_Plug_USB2.0, Q1 DMG3415U-7, SW1 RESET, SW2 ON, SW3 SW_Push, SW4 SW_Push, U1 W25Q16JV, U2 AP2112K-3.3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

Commit message: add label fboot
Parts:
- added kibuzzard-6537FB4E: G***, kibuzzard-6537FB4E, B.Cu at (112.0, 88.9)
