File: hardware/ESP32-S3/BugCON_2023.kicad_sch (KiCad schematic)
At the start: 32 parts, among them J1 Conn_01x04_Pin, J3 Conn_01x02, J4 Conn_01x01_Pin, J5 Conn_01x01_Pin, J6 SERIAL, P1 USB_C_Plug_USB2.0, Q1 DMG3415U-7, SW1 RESET, SW2 GPIO, SW3 ON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

Commit message: Change_Neopixels
Parts:
- removed D2, D3, D4, D6: WS2812B_Mini_X2, FootprintsB:LED-SMD_4P-L3.5-W3.5-TL_WS2812B-1, symbol LED:WS2812B
- added D2 (x4): WS2812B, FootprintsB:LED-SMD_4P-L3.5-W3.5-TL_WS2812B, symbol LED:WS2812B
Connections:
- net +3V3: now also D2.1 (VDD), D2.1 (VDD), D2.1 (VDD), D2.1 (VDD)
- net GND: now also D2.3 (VSS), D2.3 (VSS), D2.3 (VSS), D2.3 (VSS)
- net at R9.2: now also D2.4 (DIN)
- new net: D2.2 (DOUT), D2.4 (DIN) (x3)
